File: kikad_project/kikad_project.kicad_pcb (KiCad board)
At the start: 2 copper layers, 100 x 110 mm, 50 parts, among them IC1 HCPL-2531, IC2 HCPL-2531, IC3 HCPL-2531, J1 236-102, J10 236-104, J11 236-104, J12 236-744, J13 236-102, J14 236-102, J15 236-102, J16 236-102, J17 236-744, J18 236-102, J2 236-104, J3 236-102, J4 236-102, J5 236-744, J6 236-102, J7 236-102, J8 236-744, J9 236-102, Q2 IRF5305PbF, U1 NRF24L01_Breakout, U12 CD40109BE, U2 STM32F103C8T6, U3 L7805, U4 L7805, X1 3522-2

Commit message: PCB ready
Parts:
- moved J14 13.4 mm to (9.62, 28.6)
- moved J13 12.1 mm to (9.61, 15.9)
- moved C9 7.50 mm to (24.1, 5.08), turned to 180 degrees
- moved U2 3.73 mm to (42.8, 27.8)
- moved H3 1.27 mm to (92.7, 101.6)
- moved H2 1.27 mm to (7.62, 6.35)
- moved C8 0.73 mm to (21.1, 12.7), turned to 180 degrees
- moved U1 0.73 mm to (27.9, 3.27)
- moved J3 0.09 mm to (53.4, 100.5)
- moved J9 0.08 mm to (28.0, 100.5)
Connections:
- U2 pad 17: WHEEL_RIGHT_PWM -> DISK_PWM
- U2 pad 19: DISK_PWM -> WHEEL_RIGHT_PWM
Routing:
- net VCC: track 40.7 -> 173.6 mm
- net +24V: track 118.1 -> 2.03 mm
- net +3.3V: track 0.00 -> 75.7 mm
- net WHEEL_LEFT_PWM: track 0.00 -> 60.8 mm
- net OPT_END_DISK: track 0.00 -> 56.5 mm
- net PA9: track 0.00 -> 47.9 mm
- net DISK_PWM: track 0.00 -> 47.0 mm
- net OPT_END_WHEEL_LEFT: track 0.00 -> 45.4 mm
- net PA15: track 0.00 -> 39.8 mm
- net Net-(U12-E): track 0.00 -> 38.4 mm
- net PB3: track 0.00 -> 36.6 mm
- net PB5: track 0.00 -> 35.3 mm
- net PA10: track 0.00 -> 35.3 mm
- net PB4: track 0.00 -> 34.7 mm
- net OPT_END_WHEEL_RIGHT: track 0.00 -> 33.9 mm
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- added copper zone on F.Cu, net +24V
- added copper zone on B.Cu, net GND
