File: schemas/robot/kikad_project/kikad_project.kicad_pcb (KiCad board)
At the start: 2 copper layers, 100 x 110 mm, 50 parts, among them IC1 HCPL-2531, IC2 HCPL-2531, IC3 HCPL-2531, J1 236-102, J10 236-104, J11 236-104, J12 236-744, J13 236-102, J14 236-102, J15 236-102, J16 236-102, J17 236-744, J18 236-102, J2 236-104, J3 236-102, J4 236-102, J5 236-744, J6 236-102, J7 236-102, J8 236-744, J9 236-102, Q2 IRF5305PbF, U1 NRF24L01_Breakout, U12 CD40109BE, U2 STM32F103C8T6, U3 L7805, U4 L7805, X1 3522-2

Commit message: small edits to robot PCB schema and pcb layout
Parts:
- moved C7 3.14 mm to (80.3, 83.4)
- moved D1 3.14 mm to (75.3, 88.2)
- moved D3 3.14 mm to (90.5, 80.8)
- moved Q2 3.14 mm to (80.3, 88.4)
- moved R1 3.14 mm to (85.4, 83.4)
- moved J17 0.75 mm to (89.4, 66.9)
- moved J16 0.63 mm to (90.4, 60.6)
- moved J1 0.51 mm to (79.3, 100.5)
- moved J8 0.50 mm to (89.4, 48.4)
- moved J7 0.38 mm to (90.4, 42.1)
- moved J15 0.38 mm to (66.5, 100.5)
- moved J10 0.35 mm to (9.60, 69.9)
- moved J3 0.25 mm to (53.7, 100.5)
- moved J11 0.24 mm to (9.60, 47.1)
- moved J5 0.23 mm to (89.4, 30.0)
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Connections:
- IC1 pad 1: VCC -> DISK_PWM
- IC1 pad 2: DISK_PWM -> GND
- IC1 pad 3: DISK_DIR -> GND
- IC1 pad 4: GND -> DISK_DIR
- IC2 pad 1: VCC -> WHEEL_LEFT_PWM
- IC2 pad 2: WHEEL_LEFT_PWM -> GND
- IC2 pad 3: WHEEL_LEFT_DIR -> GND
- IC2 pad 4: GND -> WHEEL_LEFT_DIR
- IC3 pad 1: VCC -> WHEEL_RIGHT_PWM
- IC3 pad 2: WHEEL_RIGHT_PWM -> GND
- IC3 pad 3: WHEEL_RIGHT_DIR -> GND
- IC3 pad 4: GND -> WHEEL_RIGHT_DIR
- U2 pad 14: WHEEL_RIGHT_DIR -> DISK_DIR
- U2 pad 16: DISK_DIR -> WHEEL_RIGHT_DIR
Routing:
- net VCC: track 172.7 -> 141.7 mm
- net GND: track 29.2 -> 1.56 mm
- net DISK_DIR: track 50.7 -> 44.7 mm
- net DISK_PWM: track 47.0 -> 41.7 mm
- net WHEEL_LEFT_DIR: track 64.1 -> 59.1 mm
- net WHEEL_LEFT_PWM: track 60.8 -> 55.7 mm
- net WHEEL_RIGHT_PWM: track 75.1 -> 71.6 mm
- net WHEEL_RIGHT_DIR: track 76.8 -> 73.5 mm
- net Net-(Q2-S): track 19.2 -> 17.5 mm

Commit message: small changes to the PCB layout
Connections:
- H1 pad 1: GND -> unconnected-(H1-Pad1)
- H2 pad 1: GND -> unconnected-(H2-Pad1)
- H3 pad 1: GND -> unconnected-(H3-Pad1)
Routing:
- net unconnected-(H3-Pad1): track 0.00 -> 1.56 mm
- net GND: track 1.56 -> 0.00 mm
Changed lines of the file:
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@@
       (drillshape 0)
       (scaleselection 1)
-      (outputdirectory "gerber_files/")
+      (outputdirectory "production_files/")
     )
   )
@@
   (net 60 "unconnected-(U2-PB11-Pad22)")
   (net 61 "/BAT_SW")
+  (net 62 "unconnected-(H1-Pad1)")
+  (net 63 "unconnected-(H2-Pad1)")
+  (net 64 "unconnected-(H3-Pad1)")
   (footprint "236-102:CONN_236-102_WAG" (layer "F.Cu")
     (at 28.0349 100.480001)
@@
       (stroke (width 0.05) (type solid)) (fill none) (layer "F.CrtYd"))
     (pad "1" thru_hole circle (at 0 0) (size 6.4 6.4) (drill 3.2) (layers "*.Cu" "*.Mask")
-      (net 2 "GND") (pinfunction "1") (pintype "input"))
+      (net 63 "unconnected-(H2-Pad1)") (pinfunction "1") (pintype "input"))
   )
   (footprint "Capacitor_THT:C_Axial_L5.1mm_D3.1mm_P7.50mm_Horizontal" (layer "F.Cu")
@@
       (stroke (width 0.05) (type solid)) (fill none) (layer "F.CrtYd"))
     (pad "1" thru_hole circle (at 0 0) (size 6.4 6.4) (drill 3.2) (layers "*.Cu" "*.Mask")
-      (net 2 "GND") (pinfunction "1") (pintype "input"))
+      (net 62 "unconnected-(H1-Pad1)") (pinfunction "1") (pintype "input"))
   )
   (footprint "236-102:CONN_236-102_WAG" (layer "F.Cu")
@@
       (stroke (width 0.05) (type solid)) (fill none) (layer "F.CrtYd"))
     (pad "1" thru_hole circle (at 0 0) (size 6.4 6.4) (drill 3.2) (layers "*.Cu" "*.Mask")
-      (net 2 "GND") (pinfunction "1") (pintype "input"))
+      (net 64 "unconnected-(H3-Pad1)") (pinfunction "1") (pintype "input"))
   )
   (footprint "Capacitor_THT:C_Axial_L5.1mm_D3.1mm_P7.50mm_Horizontal" (layer "F.Cu")
@@
   (segment (start 6.63 60.03) (end 6.63 66.9) (width 0.5) (layer "F.Cu") (net 1))
   (segment (start 9.6 57.06) (end 6.63 60.03) (width 0.5) (layer "F.Cu") (net 1))
-  (segment (start 92.88 100.5) (end 93.98 101.6) (width 0.25) (layer "B.Cu") (net 2))
   (segment (start 34.29 91.44) (end 33.02 91.44) (width 0.5) (layer "F.Cu") (net 3))
   (segment (start 38.1 87.63) (end 34.29 91.44) (width 0.5) (layer "F.Cu") (net 3))
@@
   (segment (start 52.19 20.81) (end 52.19 18.27) (width 0.5) (layer "F.Cu") (net 44))
   (segment (start 79.3249 100.480001) (end 71.4949 100.480001) (width 3) (layer "F.Cu") (net 51))
+  (segment (start 92.88 100.5) (end 93.98 101.6) (width 0.25) (layer "B.Cu") (net 64))
   (zone (net 4) (net_name "+24V") (layer "F.Cu") (hatch edge 0.5)
     (priority 1)

Commit message: PCB edit + other minor changes
Parts:
- added REF**: ELSYS-LOGO, Library:ELSYS-LOGO, F.Cu at (24.8, 97.5)
- added REF**: MY-LOGO, Library:MY-LOGO, F.Cu at (55.4, 66.8)
- C10, C11, C12: value 100uF -> 100nF
- J12, J17, J5, J8: value 236-744 -> 236-401
- Q1: renamed from Q2; value IRF5305PbF -> IXTP120P065T
- R2, R3, R4: value 6.8МR -> 680R
- moved U12 0.19 mm to (57.4, 10.8)
- moved U2 0.14 mm to (42.9, 27.8)
Connections:
- net PA15 renamed NRF24L01_CSN
- U1 pad 3: PA10 -> NRF24L01_CE
- U1 pad 8: PA9 -> NRF24L01_IRQ
- U2 pad 27: unconnected-(U2-PB14-Pad27) -> HAND_END_RIGHT
- U2 pad 28: HAND_END_RIGHT -> HAND_END_LEFT
- U2 pad 29: HAND_END_LEFT -> unconnected-(U2-PA8-Pad29)
- U2 pad 30: PA9 -> unconnected-(U2-PA9-Pad30)
- U2 pad 31: PA10 -> NRF24L01_IRQ
- U2 pad 32: unconnected-(U2-PA11-Pad32) -> NRF24L01_CE
Routing:
- net NRF24L01_IRQ: track 0.00 -> 49.3 mm
- net PA9: track 48.2 -> 0.00 mm
- net NRF24L01_CE: track 0.00 -> 36.4 mm
- net PA10: track 35.3 -> 0.00 mm
- net WHEEL_LEFT_PWM: track 55.7 -> 57.5 mm
- net DISK_PWM: track 41.7 -> 43.5 mm
- net HAND_END_RIGHT: track 20.0 -> 19.0 mm
- net HAND_END_LEFT: track 32.3 -> 31.3 mm
- net NRF24L01_CSN: track 39.8 -> 40.3 mm

Commit message: robot schema edit
Parts:
- removed the REF** at (55.4, 66.8)
- added RN1: R_Network06, Resistor_THT:R_Array_SIP7, F.Cu at (77.0, 47.9)
- added RN2: R_Pack06_SIP, Resistor_THT:R_Array_SIP12, F.Cu at (59.1, 47.9)
- C10, C11, C12: footprint Capacitor_THT:CP_Radial_D5.0mm_P2.00mm -> Capacitor_THT:C_Rect_L4.6mm_W3.8mm_P2.50mm_MKS02_FKP02
- C2, C3, C4, C6, C7, C9: footprint Capacitor_THT:C_Axial_L5.1mm_D3.1mm_P7.50mm_Horizontal -> Capacitor_THT:C_Rect_L4.6mm_W3.8mm_P2.50mm_MKS02_FKP02
- moved REF** 87.8 mm to (78.9, 28.5)
- moved IC1 17.7 mm to (66.1, 51.7)
- moved IC2 17.6 mm to (66.1, 64.2)
- moved IC3 17.5 mm to (66.1, 76.7)
- moved C5 8.96 mm to (47.0, 80.8)
- moved C6 8.96 mm to (51.5, 82.0)
- moved U4 8.96 mm to (46.4, 88.5)
- moved C4 8.93 mm to (56.6, 88.6)
- moved C1 7.82 mm to (32.3, 74.2)
- moved C3 7.82 mm to (25.2, 92.0)
- moved U3 7.82 mm to (30.3, 81.8)
- moved C2 7.82 mm to (37.9, 76.7)
- moved L1 7.82 mm to (35.4, 88.2)
- moved C10 5.25 mm to (27.1, 62.0), turned to 180 degrees
- moved C12 5.10 mm to (27.1, 52.1), turned to 180 degrees
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Connections:
- net Net-(IC1-V01) renamed /IC1_VO1
- net Net-(IC1-V02) renamed /IC1_VO2
- net Net-(IC2-V01) renamed /IC2_VO1
- net Net-(IC2-V02) renamed /IC2_VO2
- net Net-(IC3-V01) renamed /IC3_VO1
- net Net-(IC3-V02) renamed /IC3_VO2
- IC1 pad 1: DISK_PWM -> /IC1_VF1+
- IC1 pad 4: DISK_DIR -> /IC1_VF2+
- IC2 pad 1: WHEEL_LEFT_PWM -> /IC2_VF1+
- IC2 pad 4: WHEEL_LEFT_DIR -> /IC2_VF2+
- IC3 pad 1: WHEEL_RIGHT_PWM -> /IC3_VF1+
- IC3 pad 4: WHEEL_RIGHT_DIR -> /IC3_VF2+
- Q1 pad 2: +24V -> Net-(Q1-S)
- Q1 pad 3: Net-(Q1-S) -> +24V
Routing:
- net DISK_PWM: track 43.5 -> 73.4 mm
- net WHEEL_LEFT_PWM: track 57.5 -> 82.9 mm
- net /IC3_VO2: track 9.99 -> 34.0 mm
- net /IC1_VO2: track 20.2 -> 43.4 mm
- net /IC3_VO1: track 12.0 -> 35.0 mm
- net /IC1_VO1: track 22.6 -> 45.6 mm
- net WHEEL_RIGHT_PWM: track 71.5 -> 93.9 mm
- net /IC2_VO1: track 16.9 -> 37.6 mm
- net DISK_DIR: track 44.6 -> 65.2 mm
- net /IC2_VO2: track 15.1 -> 35.1 mm
- net WHEEL_LEFT_DIR: track 58.9 -> 75.0 mm
- net WHEEL_RIGHT_DIR: track 73.4 -> 86.1 mm
- net /IC3_VF2+: track 0.00 -> 6.05 mm
- net VCC: track 141.7 -> 136.9 mm
- net Net-(Q1-S): track 17.5 -> 21.8 mm
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